Commit message: Fix issues with Robot Xacro file and also modify world model

File: src/my_robot/urdf/my_robot.xacro (robot description, xacro)
@@ -8,12 +8,4 @@
     <child link="chassis" />
   </joint>
-  <!--
-  <link name="odom"></link>
-  <joint name="odom" type="fixed">
-    <origin xyz="0 0 0" rpy=" 0 0 0"/>
-    <parent link="odom"/>
-    <child link="chassis" />
-  </joint>
-  -->
   <link name='chassis'>
     <pose>0 0 0.1 0 0 0</pose>
@@ -30,5 +22,6 @@
       <origin xyz="0 0 0" rpy=" 0 0 0"/>
       <geometry>
-        <box size=".4 .2 .1"/>
+        <!--<box size=".4 .2 .1"/>-->
+        <cylinder length="0.1" radius="0.2"/>
       </geometry>
     </collision>
@@ -36,5 +29,6 @@
       <origin xyz="0 0 0" rpy=" 0 0 0"/>
       <geometry>
-        <box size=".4 .2 .1"/>
+        <!--<box size=".4 .2 .1"/>-->
+        <cylinder length="0.1" radius="0.2"/>
       </geometry>
     </visual>
@@ -64,8 +58,8 @@
     </visual>
   </link>
-  <gazebo reference="chassis">
+   <gazebo reference="chassis">
     <material>Gazebo/Red</material>
   </gazebo>
-  <link name="link_right_wheel">
+  <link name="left_wheel">
     <inertial>
       <mass value="5"/>
@@ -73,5 +67,5 @@
       <inertia ixx="0.1" ixy="0" ixz="0" iyy="0.1" iyz="0" izz="0.1"/>
     </inertial>
-    <collision name="link_right_wheel_collision">
+    <collision name="left_wheel_collision">
       <origin rpy="0 1.5707 1.5707" xyz="0 0 0" />
       <geometry>
@@ -79,5 +73,36 @@
       </geometry>
     </collision>
-    <visual name="link_right_wheel_visual">
+    <visual name="left_wheel_visual">
+      <origin rpy="0 1.5707 1.5707" xyz="0 0 0"/>
+      <geometry>
+        <cylinder length="0.05" radius="0.1"/>
+      </geometry>
+    </visual>
+  </link>
+  <!--   Joint for left wheel  -->
+  <joint name="left_wheel_hinge" type="continuous">
+    <origin rpy="0 0 0" xyz="0 0.15 0"/>
+    <child link="left_wheel" />
+    <parent link="chassis"/>
+    <axis rpy="0 0 0" xyz="0 1 0"/>
+    <limit effort="10000" velocity="1000"/>
+    <joint_properties damping="1.0" friction="1.0" />
+  </joint>
+  <gazebo reference="left_wheel">
+    <material>Gazebo/Green</material>
+  </gazebo>
+  <link name="right_wheel">
+    <inertial>
+      <mass value="5"/>
+      <origin rpy="0 1.5707 1.5707" xyz="0 0 0"/>
+      <inertia ixx="0.1" ixy="0" ixz="0" iyy="0.1" iyz="0" izz="0.1"/>
+    </inertial>
+    <collision name="right_wheel_collision">
+      <origin rpy="0 1.5707 1.5707" xyz="0 0 0" />
+      <geometry>
+        <cylinder length="0.05" radius="0.1"/>
+      </geometry>
+    </collision>
+    <visual name="right_wheel_visual">
       <origin rpy="0 1.5707 1.5707" xyz="0 0 0"/>
       <geometry>
@@ -87,7 +112,7 @@
   </link>
   <!--   Joint for right wheel  -->
-  <joint name="joint_right_wheel" type="continuous">
-    <origin rpy="0 0 0" xyz="0 0.15 0"/>
-    <child link="link_right_wheel" />
+  <joint name="right_wheel_hinge" type="continuous">
+    <origin rpy="0 0 0" xyz="0 -0.15 0"/>
+    <child link="right_wheel" />
     <parent link="chassis"/>
     <axis rpy="0 0 0" xyz="0 1 0"/>
@@ -95,98 +120,65 @@
     <joint_properties damping="1.0" friction="1.0" />
   </joint>
-  <gazebo reference="link_right_wheel">
-    <material>Gazebo/Green</material>
-  </gazebo>
-  <link name="link_left_wheel">
-    <inertial>
-      <mass value="5"/>
-      <origin rpy="0 1.5707 1.5707" xyz="0 0 0"/>
-      <inertia ixx="0.1" ixy="0" ixz="0" iyy="0.1" iyz="0" izz="0.1"/>
-    </inertial>
-    <collision name="link_left_wheel_collision">
-      <origin rpy="0 1.5707 1.5707" xyz="0 0 0" />
-      <geometry>
-        <cylinder length="0.05" radius="0.1"/>
-      </geometry>
-    </collision>
-    <visual name="link_left_wheel_visual">
-      <origin rpy="0 1.5707 1.5707" xyz="0 0 0"/>
-      <geometry>
-        <cylinder length="0.05" radius="0.1"/>
-      </geometry>
-    </visual>
-  </link>
-    <!--   Joint for left wheel  -->
-  <joint name="joint_left_wheel" type="continuous">
-    <origin rpy="0 0 0" xyz="0 -0.15 0"/>
-    <child link="link_left_wheel" />
-    <parent link="chassis"/>
-    <axis rpy="0 0 0" xyz="0 1 0"/>
-    <limit effort="10000" velocity="1000"/>
-    <joint_properties damping="1.0" friction="1.0" />
-  </joint>
-  <gazebo reference="link_left_wheel">
-    <material>Gazebo/Green</material>
-  </gazebo>
-  <link name="camera">
+<gazebo reference="right_wheel">
+<material>Gazebo/Green</material>
+</gazebo>
+<link name='camera'>
+    <pose>0 0 0 0 0 0</pose>
     <inertial>
       <mass value="0.1"/>
-      <origin rpy="0 0 0" xyz="0 0 0"/>
-      <box_inertia m="0.1" x="0.05" y="0.05" z="0.05"/>
-      <inertia ixx="1e-6" ixy="0" ixz="0" iyy="1e-6" iyz="0" izz="1e-6"/>
+      <origin xyz="0.0 0 0" rpy=" 0 0 0"/>
+      <inertia
+          ixx="1e-6" ixy="0" ixz="0" iyy="1e-6" iyz="0" izz="1e-6"
+      />
     </inertial>
-    <collision name="camera_collision">
-      <origin rpy="0 0 0" xyz="0 0 0" />
+    <collision name='camera_collision'>
+      <origin xyz="0 0 0" rpy=" 0 0 0"/>
       <geometry>
         <box size="0.05 0.05 0.05"/>
       </geometry>
     </collision>
-    <visual name="camera_visual">
-      <origin rpy="0 0 0" xyz="0 0 0"/>
+    <visual name='camera_visual'>
+      <origin xyz="0 0 0" rpy=" 0 0 0"/>
       <geometry>
         <box size="0.05 0.05 0.05"/>
       </geometry>
     </visual>
-  </link>
-  <gazebo reference="camera">
-    <material>Gazebo/Blue</material>
-  </gazebo>
-  <!--   Joint for camera  -->
+</link>
   <joint name="camera_joint" type="fixed">
-    <origin rpy="0 0 0" xyz="0.2 0 0"/>
+    <origin xyz="0.2 0 0" rpy="0 0 0" />
+    <parent link="chassis"/>
     <child link="camera" />
-    <parent link="chassis"/>
-    <axis rpy="0 0 0" xyz="0 1 0"/>
-    <limit effort="10000" velocity="1000"/>
-    <joint_properties damping="1.0" friction="1.0" />
+    <axis xyz="0 1 0" rpy="0 0 0"/>
   </joint>
-  <!--   Link for Lidar  -->
-   <link name="hokuyo">
+<gazebo reference="camera">
+  <material>Gazebo/Blue</material>
+</gazebo>
+ <link name='hokuyo'>
+    <pose>0 0 0 0 0 0</pose>
     <inertial>
       <mass value="1e-5"/>
-      <origin rpy="0 0 0" xyz="0 0 0"/>
-      <inertia ixx="1e-6" ixy="0" ixz="0" iyy="1e-6" iyz="0" izz="1e-6"/>
+      <origin xyz="0.0 0 0" rpy=" 0 0 0"/>
+      <inertia
+          ixx="1e-6" ixy="0" ixz="0" iyy="1e-6" iyz="0" izz="1e-6"
+      />
     </inertial>
-    <collision name="hokuyo_collision">
-      <origin rpy="0 0 0" xyz="0 0 0" />
+    <collision name='hokuyo_collision'>
+      <origin xyz="0 0 0" rpy=" 0 0 0"/>
       <geometry>
         <box size="0.1 0.1 0.1"/>
       </geometry>
     </collision>
-    <visual name="hokuyo_visual">
-      <origin rpy="0 0 0" xyz="0 0 0"/>
+    <visual name='hokuyo_visual'>
+      <origin xyz="0 0 0" rpy=" 0 0 0"/>
       <geometry>
         <mesh filename="package://my_robot/meshes/hokuyo.dae"/>
       </geometry>
     </visual>
-  </link>
-  <!--   Joint for lidar  -->
+</link>
   <joint name="hokuyo_joint" type="fixed">
-    <origin rpy="0 0 0" xyz="0.15 0 0.1"/>
-    <child link="hokuyo" />
-    <parent link="chassis"/>
-    <axis rpy="0 0 0" xyz="0 1 0"/>
-    <limit effort="10000" velocity="1000"/>
-    <joint_properties damping="1.0" friction="1.0" />
+  <origin xyz="0.15 0 0.1" rpy="0 0 0" />
+  <parent link="chassis"/>
+  <child link="hokuyo" />
+  <axis xyz="0 1 0" rpy="0 0 0"/>
   </joint>
 </robot>

Commit message: Give a little offset to chassis

File: src/my_robot/urdf/my_robot.xacro (robot description, xacro)
@@ -20,14 +20,12 @@
     </inertial>
     <collision name='collision'>
-      <origin xyz="0 0 0" rpy=" 0 0 0"/>
+      <origin xyz="0 0 0.025" rpy=" 0 0 0"/>
       <geometry>
-        <!--<box size=".4 .2 .1"/>-->
         <cylinder length="0.1" radius="0.2"/>
       </geometry>
     </collision>
     <visual name='chassis_visual'>
-      <origin xyz="0 0 0" rpy=" 0 0 0"/>
+      <origin xyz="0 0 0.025" rpy=" 0 0 0"/>
       <geometry>
-        <!--<box size=".4 .2 .1"/>-->
         <cylinder length="0.1" radius="0.2"/>
       </geometry>
